File: main/picoTracker.kicad_sch (KiCad schematic)
At the start: 104 parts, among them IC1 XC6206P332MR, IC2 XC6206P332MR, IC3 BQ24232HRGTR, IC4 W25Q128JVS, IC5 PCM5102A, IC6 RP2040, IC7 TPA6139A2RGTR, IC8 H11L1, J1 5027740891, J2 USB_C_Receptacle_USB2.0, J3 Conn_01x02, J4 Conn_01x10, J5 Conn_01x18, J6 Headphones, J7 Conn_02x03_Odd_Even, J8 MIDI Out, J9 MIDI In, SW1 MS-22D28-G020, SW2 SW_SPST, Y1 12MHz 20pF ±10ppm

Commit message: picoTracker PCB v2.1 and picoTrackerKeypad PCB v2.0
Parts:
- removed C27, C29, C31, C39: 10uF, Capacitor_Tantalum_SMD:CP_EIA-3216-18_Kemet-A, symbol Device:C_Polarized
- removed C41: 2.2uF, Capacitor_SMD:C_0603_1608Metric, symbol Device:C
- removed C42, C43, C44: 1uF, Capacitor_SMD:C_0603_1608Metric, symbol Device:C
- removed IC3: BQ24232HRGTR, project:QFN50P300X300X100-17N-D, symbol BQ24232HRGTR:BQ24232HRGTR
- removed IC7: TPA6139A2RGTR, project:QFN50P300X300X100-17N-D, symbol TPA6139A2RGTR:TPA6139A2RGTR
- removed J1: 5027740891, project:MOLEX_5027740891, symbol Molex SD inverted push-push:5027740891
- removed J3: Conn_01x02, project:PinHeader_1x02_P2.54mm_Vertical, symbol Connector_Generic:Conn_01x02
- removed J4: Conn_01x10, project:PinHeader_1x10_P2.54mm_Vertical, symbol Connector_Generic:Conn_01x10
- removed J5: Conn_01x18, project:QD-TFT2803, symbol Connector_Generic:Conn_01x18
- removed J6: Headphones, project:PJ327C4A, symbol PJ-327C-4A:PJ-327C-4A
- removed J7: Conn_02x03_Odd_Even, project:PinHeader_2x03_P2.54mm_Vertical, symbol Connector_Generic:Conn_02x03_Odd_Even
- removed R17, R18: 100k, Resistor_SMD:R_0603_1608Metric, symbol Device:R
- removed R19: 82k, Resistor_SMD:R_0805_2012Metric, symbol Device:R
- removed R7: 4.3k, Resistor_SMD:R_0603_1608Metric, symbol Device:R
- removed TP1: VBAT, TestPoint:TestPoint_Pad_D1.0mm, symbol Connector:TestPoint
- removed TP2: TestPoint, TestPoint:TestPoint_Pad_D1.0mm, symbol Connector:TestPoint
- removed TP3: VCHR, TestPoint:TestPoint_Pad_D1.0mm, symbol Connector:TestPoint
- removed TP4: 3.3VA, TestPoint:TestPoint_Pad_D1.0mm, symbol Connector:TestPoint
- removed TP5: VBUS, TestPoint:TestPoint_Pad_D1.0mm, symbol Connector:TestPoint
- removed TP6: GND, TestPoint:TestPoint_Pad_D1.0mm, symbol Connector:TestPoint
- added C27, C29, C31: 10uF, Capacitor_SMD:C_0603_1608Metric, symbol Device:C
- added C47, C49, C57: 1uF, Capacitor_SMD:C_0603_1608Metric, symbol Device:C
- added C48: 2.2uF, Capacitor_SMD:C_0603_1608Metric, symbol Device:C
- added D2: LED, LED_SMD:LED_0603_1608Metric, symbol Device:LED
- added IC3: TPA6139A2RGTR, project:QFN50P300X300X100-17N-D, symbol TPA6139A2RGTR:TPA6139A2RGTR
- added J1: Conn_01x03, project:CONN_S3B-ZR-SM4A-TFLFSN_JST, symbol Connector_Generic:Conn_01x03
- added J10: FPC-05FB-40PH20, project:FPC_40-flap, symbol Connector_Generic:Conn_01x40
- added J3: Conn_02x10_Counter_Clockwise, Connector_Hirose:Hirose_DF12_DF12C3.0-20DS-0.5V_2x10_P0.50mm_Vertical, symbol Connector_Generic:Conn_02x10_Counter_Clockwise
- added J4: Micro_SD_Card, project:Xunpu_TF-115_microSD, symbol Connector:Micro_SD_Card
- added J5: Headphones, project:PJ327C4A, symbol PJ-327C-4A:PJ-327C-4A
- added R27: 1k, Resistor_SMD:R_0603_1608Metric, symbol Device:R
- added R29: 560, Resistor_SMD:R_0603_1608Metric, symbol Device:R
- added R4: 82k, Resistor_SMD:R_0805_2012Metric, symbol Device:R
- added U1: AP2502KTR-G1, project:SOT23-6_DIO, symbol AP2502KTR-G1:AP2502KTR-G1
- added U2: BQ24074RGT, Package_DFN_QFN:VQFN-16-1EP_3x3mm_P0.5mm_EP1.6x1.6mm, symbol Battery_Management:BQ24074RGT
- C22: value 10uF -> 2.2uF; LCSC C19702 -> C23630
- C40: value 2.2uF -> 10uF; LCSC C23630 -> C19702
- D1: JLCPCB Rotation Offset (none) -> 0
- H1, H2, H3, H4: footprint MountingHole:MountingHole_2.2mm_M2 -> MountingHole:MountingHole_3.2mm_M3
- IC6, IC8: JLCPCB Rotation Offset (none) -> -90
- J2: JLCPCB Position Offset (none) -> 0,1.3125
- J8, J9: JLCPCB Position Offset (none) -> 1.905,0.125; JLCPCB Rotation Offset (none) -> 90
- R1, R8: value 10k -> 1k; LCSC C25804 -> C21190
- R12: now not fitted
- R2: value 3k -> 100k; LCSC C4211 -> C25803
- R22: LCSC C25905 -> C1111
- R3: value 10k -> 100k; LCSC C25804 -> C25803
Connections:
- net VBAT is gone; now on net LINE_OUT_R: C22.1
- net +3.3VA: now also C40.1, C29.1, C49.1, IC3.4 (~{MUTE}), IC3.9 (VDD)
- net +3V3: now also C27.1, J10.33 (Pin_33), J10.39 (Pin_39), J10.40 (Pin_40), J10.6 (Pin_6), J10.7 (Pin_7), J3.1 (Pin_1), J4.4 (VDD)
- net BAT: now also R2.2, R3.1
- net DISPLAY_CS: now also J10.9 (Pin_9)
- net DISPLAY_DC: now also J10.11 (Pin_11)
- net DISPLAY_MOSI: now also J10.13 (Pin_13)
- net DISPLAY_RST: now also J10.15 (Pin_15)
- net DISPLAY_SCK: now also J10.10 (Pin_10)
- net GND: now also C40.2, R3.2, C27.2, C29.2, C31.2, C49.2, C57.2, IC3.10 (GND_3), IC3.17 (EP), IC3.2 (GND_1), IC3.3 (GND_2), J1.1 (Pin_1), J10.12 (Pin_12), J10.16 (Pin_16), J10.17 (Pin_17), J10.18 (Pin_18), J10.19 (Pin_19), J10.20 (Pin_20), J10.21 (Pin_21), J10.22 (Pin_22), J10.23 (Pin_23), J10.24 (Pin_24), J10.25 (Pin_25), J10.26 (Pin_26), J10.27 (Pin_27), J10.28 (Pin_28), J10.29 (Pin_29), J10.30 (Pin_30), J10.31 (Pin_31), J10.32 (Pin_32), J10.37 (Pin_37), J10.38 (Pin_38), J10.5 (Pin_5), J3.11 (Pin_11), J4.6 (VSS), J4.9 (SHIELD), J5.1, R27.1, R29.1, R4.2, U1.2 (GND), U2.17 (VSS), U2.4 (~{CE}), U2.6 (EN1), U2.8 (VSS); no longer C22.2, R2.1, R8.1
- net LINE_OUT_L: now also C48.1
- net LINE_OUT_R: no longer C40.1
- net OUT_HP_L: now also IC3.12 (OUT_R), J5.2
- net OUT_HP_R: now also IC3.1 (OUT_L), J5.3
- net SD_CLK: now also J4.5 (CLK)
- net SD_CMD: now also J4.3 (CMD)
- net SD_D0: now also J4.7 (DAT0)
- net SD_D1: now also J4.8 (DAT1)
- net SD_D2: now also J4.1 (DAT2)
- net SD_D3: now also J4.2 (DAT3/CD)
- net SWCLK: now also J3.16 (Pin_16)
- net SWDIO: now also J3.17 (Pin_17)
- net VBUS: now also C57.1, U2.13 (IN); no longer C13.1
- net VCHR1: now also R8.2, U2.10 (OUT), U2.11 (OUT), U2.5 (EN2); no longer R3.2
- net VCHR2: now also R2.1
- net at C38.1, IC5.18 (LDOO): now also C31.1
- net at R1.1: now also D2.2 (A)
- net +3.3VApre: now reaches C8.1, C9.1, FB1.1, IC2.2 (VO)
- net +1V1 renamed +1.1V
- net BCK renamed DAC_I2S_BCK
- net DIN renamed DAC_I2S_DATA
- net LRCK renamed DAC_I2S_LRCK
- net SCK renamed DISPLAY_PWM
- net DISPLAY_PWM: now also U1.1 (EN)
- net SW_A renamed INPUT_ENTER
- net INPUT_ENTER: now also J3.8 (Pin_8)
- net SW_B renamed INPUT_EDIT
- net INPUT_EDIT: now also J3.7 (Pin_7)
- net SW_DOWN renamed INPUT_DOWN
- net INPUT_DOWN: now also J3.3 (Pin_3)
- net SW_LEFT renamed INPUT_LEFT
- net INPUT_LEFT: now also J3.2 (Pin_2)
- net SW_LT renamed INPUT_ALT
- net INPUT_ALT: now also J3.6 (Pin_6)
- net SW_PLAY renamed INPUT_PLAY
- net INPUT_PLAY: now also J3.10 (Pin_10)
- net SW_RIGHT renamed INPUT_RIGHT
- net INPUT_RIGHT: now also J3.4 (Pin_4)
- net SW_RT renamed INPUT_NAV
- net INPUT_NAV: now also J3.9 (Pin_9)
- net SW_UP renamed INPUT_UP
- net INPUT_UP: now also J3.5 (Pin_5)
- net VOL renamed DISPLAY_MISO
- net DISPLAY_MISO: now also J10.14 (Pin_14)
- net i2c0_SCL renamed DEBUG_RX
- net DEBUG_RX: now also J3.19 (Pin_19)
- net i2c0_SDA renamed DEBUG_TX
- net DEBUG_TX: now also J3.18 (Pin_18)
- new net: IC3.11 (GAIN), R4.1
- new net: C48.2, IC3.13 (-IN_R)
- new net: C22.2, IC3.16 (-IN_L)
- new net: C13.1, IC3.5 (VSS)
- new net: C47.1, IC3.6 (CN)
- new net: C47.2, IC3.8 (CP)
- new net: R27.2, U2.12 (ILIM)
- new net: J1.2 (Pin_2), U2.1 (TS)
- new net: J1.3 (Pin_3), U2.2 (BAT), U2.3 (BAT)
- new net: R29.2, U2.16 (ISET)
- new net LED1-K: J10.34 (Pin_34), U1.6 (LED1)
- new net LED2-K: J10.35 (Pin_35), U1.5 (LED2)
- new net LED3-K: J10.36 (Pin_36), U1.4 (LED3)
- new net ~{CHR}: D2.1 (K), U2.9 (~{CHG})
- new net ~{PGOOD}: R8.1, U2.7 (~{PGOOD})
- no-connect marks 24 -> 25
Other:
- note added: "Battery: LIP1708 60x39x7.5 1500 - 2500mAh JST-ZH (1.5mm pitch)"
- note added: "ILIM: 1500mA"
- note added: "IM0: 0 IM1: 1 IM2: 1 - 4-wire 8-bit data serial interface"
- note added: "ISET: 1500mA"
- note added: "ITERM: unconnected - default 10% threshold"
- note added: "TMR: unconnected - default 5h"
- note removed: "en1,en2 max input current config. 500mA"
- note removed: "iterm: leave at default 10% threshold"
- moved on the sheet: C3, C4, R1
